File: DUE_PCB_V1.01/Ardumower.kicad_pcb (KiCad board)
At the start: 2 copper layers, 169.3 x 95.5 mm, 86 parts, among them J1 I2C_1, J10 Bumper Left, J11 Bumper Right, J12 P_Left, J13 P_Right, J14 Sonar_R, J15 Sonar_C, J16 Sonar_L, J17 US1, J18 US2, J19 US3, J2 I2C_2, J20 Button, J21 5V IN, J22 Remote, J23 PCB_2, J24 3.3V IN, J25 TX0/RX0, J26 TX1/RX1, J27 TX2/RX2, J28 GPS_TX/GPS_RX, J29 Motor_Right1, J3 I2C_3, J30 Motor_Right2, J31 Motor_Left1, J32 Motor_Left2, J33 Cutter_Motor, J34 ODORight1, J35 ODORight2, J36 ODOLeft1, J37 ODOLeft2, J38 ODOCutter, J4 DS3231 RTC, J5 9V IN, J6 Drop_Left, J7 Drop_Right, J8 Tilt, J9 Rain

Commit message: first test
Parts:
- removed D1: LED_DUE_3V, LED_THT:LED_D3.0mm
- removed D2: LED_DUE_5V, LED_THT:LED_D3.0mm
- removed J11: Bumper Right, Zimprich:Pin_Header_KK110_1x02_3D
- removed JP3: Buzzer OFF, Connector_PinHeader_2.54mm:PinHeader_1x02_P2.54mm_Vertical
- removed R15: 100, Resistor_THT:R_Axial_DIN0207_L6.3mm_D2.5mm_P2.54mm_Vertical
- removed R16: 220, Resistor_THT:R_Axial_DIN0207_L6.3mm_D2.5mm_P2.54mm_Vertical
- removed SP1: SPEAKER, Zimprich:Buzzer_12x9.5RM7.6
- added J39: MC33926 compatibility sense, Connector_JST:JST_XH_B4B-XH-A_1x04_P2.50mm_Vertical, F.Cu at (160.0, 115.6)
- added J40: MC33926 compatibility fault, Connector_JST:JST_XH_B4B-XH-A_1x04_P2.50mm_Vertical, F.Cu at (160.0, 123.4)
- added J41: Buzzer, Connector_JST:JST_XH_B3B-XH-A_1x03_P2.50mm_Vertical, F.Cu at (44.5, 119.4)
- J1: value I2C_1 -> I2C0_1; footprint Connector_PinHeader_2.54mm:PinHeader_1x04_P2.54mm_Vertical -> Connector_JST:JST_XH_B4B-XH-A_1x04_P2.50mm_Vertical
- J10: value Bumper Left -> Bumper; footprint Connector_PinHeader_2.54mm:PinHeader_1x02_P2.54mm_Vertical -> Connector_JST:JST_XH_B3B-XH-A_1x03_P2.50mm_Vertical
- J2: value I2C_2 -> I2C0_2; footprint Connector_PinHeader_2.54mm:PinHeader_1x04_P2.54mm_Vertical -> Connector_JST:JST_XH_B4B-XH-A_1x04_P2.50mm_Vertical
- J25: value TX0/RX0 -> Ser0
- J26: value TX1/RX1 -> Ser1
- J27: value TX2/RX2 -> Ser2
- J28: value GPS_TX/GPS_RX -> Ser3
- J3: value I2C_3 -> I2C1_1; footprint Connector_PinHeader_2.54mm:PinHeader_1x04_P2.54mm_Vertical -> Connector_JST:JST_XH_B4B-XH-A_1x04_P2.50mm_Vertical
- J4: value DS3231 RTC -> I2C1_2; footprint Connector_PinHeader_2.54mm:PinHeader_1x06_P2.54mm_Vertical -> Connector_JST:JST_XH_B4B-XH-A_1x04_P2.50mm_Vertical
- J6, J7, J8, J9: footprint Connector_PinHeader_2.54mm:PinHeader_1x03_P2.54mm_Vertical -> Connector_JST:JST_XH_B3B-XH-A_1x03_P2.50mm_Vertical
- moved J10 104.6 mm to (167.6, 20.3)
- moved J22 42.4 mm to (138.4, 54.6), turned to 270 degrees
- moved J4 42.2 mm to (83.8, 48.3), turned to 0 degrees
- moved R27 41.5 mm to (74.9, 41.9), turned to 90 degrees
- moved R9 38.7 mm to (74.9, 48.3), turned to 90 degrees
- moved J3 32.7 mm to (83.8, 39.4)
- moved R8 26.8 mm to (99.1, 49.5), turned to 90 degrees
- moved R13 23.2 mm to (99.1, 41.9), turned to 90 degrees
- moved C1 12.7 mm to (61.0, 53.3)
- moved D5 12.7 mm to (66.6, 38.9)
- moved R14 12.7 mm to (65.5, 45.7)
- moved J1 9.40 mm to (106.7, 48.3)
- moved D4 6.35 mm to (60.9, 38.9)
- moved R17 6.35 mm to (53.7, 45.6)
- moved R18 6.35 mm to (59.8, 45.6)
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Connections:
- J10 pad 2: pinBumperLeft -> pinBumperRight
- J28 pad 3: GPS_RX -> RX3
- J28 pad 4: GPS_TX -> TX3
- J30 pad 2: pinMotorRightDir -> pinMotorRight2Dir
- J32 pad 2: pinMotorLeftDir -> pinMotorLeft2Dir
- J4 pad 1: (no net) -> +3V3
- J4 pad 2: (no net) -> GND
- J4 pad 3: SCL1 -> SDA1
- J4 pad 4: SDA1 -> SCL1
- XA1 pad A0: (no net) -> pinMotorRightSense
- XA1 pad A1: (no net) -> pinMotorLeftSense
- XA1 pad A3: (no net) -> pinMotorMow2Sense
- XA1 pad A6: (no net) -> pinMotorMow1Sense
- XA1 pad D14: GPS_RX -> TX3
- XA1 pad D15: GPS_TX -> RX3
- XA1 pad D25: (no net) -> pinMotorLeftFault
- XA1 pad D26: (no net) -> pinMotorMowFault
- XA1 pad D27: (no net) -> pinMotorRightFault
- XA1 pad D40: (no net) -> pinMotorLeft2Dir
- XA1 pad D41: (no net) -> pinMotorRight2Dir

Commit message: half job
Parts:
- removed J27: Ser2, Connector_PinHeader_2.54mm:PinHeader_1x05_P2.54mm_Vertical
- removed R1, R2, R5: 1KO, Resistor_THT:R_Axial_DIN0207_L6.3mm_D2.5mm_P2.54mm_Vertical
- removed R12, R6, R7: 2KO, Resistor_THT:R_Axial_DIN0207_L6.3mm_D2.5mm_P2.54mm_Vertical
- added J11: Sonar_C, Connector_JST:JST_XH_B4B-XH-A_1x04_P2.50mm_Vertical, F.Cu at (161.3, 124.5)
- J12, J13: footprint Connector_PinHeader_2.54mm:PinHeader_1x03_P2.54mm_Vertical -> Connector_JST:JST_XH_B3B-XH-A_1x03_P2.50mm_Vertical
- J14, J16: footprint Connector_PinHeader_2.54mm:PinHeader_1x04_P2.54mm_Vertical -> Connector_JST:JST_XH_B4B-XH-A_1x04_P2.50mm_Vertical
- J15: value Sonar_C -> Ser2 ESP32; footprint Connector_PinHeader_2.54mm:PinHeader_1x04_P2.54mm_Vertical -> Connector_JST:JST_XH_B4B-XH-A_1x04_P2.50mm_Vertical
- J20: footprint Zimprich:Pin_Header_KK110_1x02_3D -> Connector_JST:JST_XH_B2B-XH-A_1x02_P2.50mm_Vertical
- J25, J26, J28: footprint Connector_PinHeader_2.54mm:PinHeader_1x05_P2.54mm_Vertical -> Connector_JST:JST_XH_B5B-XH-A_1x05_P2.50mm_Vertical
- J8: footprint Connector_JST:JST_XH_B3B-XH-A_1x03_P2.50mm_Vertical -> Connector_JST:JST_XH_B2B-XH-A_1x02_P2.50mm_Vertical
- moved J10 147.5 mm to (58.4, 119.4)
- moved J6 101.4 mm to (44.5, 109.2)
- moved J22 93.9 mm to (57.1, 101.6)
- moved J7 93.2 mm to (58.4, 109.2)
- moved J25 90.2 mm to (123.2, 39.4)
- moved J14 88.2 mm to (171.4, 119.4)
- moved J28 84.1 mm to (142.2, 48.3)
- moved J16 80.9 mm to (146.1, 119.4)
- moved J26 79.8 mm to (123.2, 48.3)
- moved R20 78.7 mm to (152.4, 97.8)
- moved R19 76.8 mm to (152.4, 92.7)
- moved R25 73.1 mm to (143.5, 73.7)
- moved R24 71.2 mm to (143.5, 86.4)
- moved R26 69.4 mm to (143.5, 67.3)
- moved R22 66.5 mm to (143.5, 80.0)
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Connections:
- J14 pad 1: +5V -> +3V3
- J14 pad 3: Net-(J14-Pad3) -> pinSonarRightEcho
- J15 pad 1: +5V -> GND
- J15 pad 2: GND -> RX2
- J15 pad 3: Net-(J15-Pad3) -> TX2
- J15 pad 4: pinSonarCenterTrigger -> +9V
- J16 pad 1: +5V -> +3V3
- J16 pad 3: Net-(J16-Pad3) -> pinSonarLeftEcho
- J25 pad 1: +3V3 -> (no net)
- J25 pad 2: GND -> (no net)
- J25 pad 3: RX0 -> (no net)
- J25 pad 4: TX0 -> (no net)
- J25 pad 5: +5V -> (no net)
- J8 pad 1: +3V3 -> GND
- J8 pad 2: GND -> pinTilt
- XA1 pad D0: RX0 -> (no net)
- XA1 pad D1: TX0 -> (no net)
