File: DUE_PCB_V1.01/Ardumower.sch (KiCad schematic (older format))
At the start: 62 parts, among them J1 I2C_1, J10 Bumper Left, J11 Bumper Right, J12 P_Left, J13 P_Right, J14 Sonar_R, J15 Sonar_C, J16 Sonar_L, J17 US1, J18 US2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

Commit message: first test
Parts:
- removed D1: LED_DUE_3V, LED_THT:LED_D3.0mm, symbol Zimprich:LED
- removed D2: LED_DUE_5V, LED_THT:LED_D3.0mm, symbol Zimprich:LED
- removed J10: Bumper Left, Connector_PinHeader_2.54mm:PinHeader_1x02_P2.54mm_Vertical, symbol Connector:Screw_Terminal_01x02
- removed J11: Bumper Right, Zimprich:Pin_Header_KK110_1x02_3D, symbol Connector:Screw_Terminal_01x02
- removed J4: DS3231 RTC, Connector_PinHeader_2.54mm:PinHeader_1x06_P2.54mm_Vertical, symbol Connector:Screw_Terminal_01x06
- removed JP3: Buzzer OFF, Connector_PinHeader_2.54mm:PinHeader_1x02_P2.54mm_Vertical, symbol Jumper:Jumper_2_Open
- removed R15: 100, Resistor_THT:R_Axial_DIN0207_L6.3mm_D2.5mm_P2.54mm_Vertical, symbol Device:R
- removed R16: 220, Resistor_THT:R_Axial_DIN0207_L6.3mm_D2.5mm_P2.54mm_Vertical, symbol Device:R
- removed SP1: SPEAKER, Zimprich:Buzzer_12x9.5RM7.6, symbol Lötpad_2,5mm:SPEAKER
- added J10: Bumper, Connector_JST:JST_XH_B3B-XH-A_1x03_P2.50mm_Vertical, symbol Connector:Screw_Terminal_01x03
- added J4: I2C1_2, Connector_JST:JST_XH_B4B-XH-A_1x04_P2.50mm_Vertical, symbol Connector:Screw_Terminal_01x04
- added J41: Buzzer, Connector_JST:JST_XH_B3B-XH-A_1x03_P2.50mm_Vertical, symbol Connector:Screw_Terminal_01x03
- D3, D4, D5: symbol Zimprich:LED -> Ardumower-rescue:LED-Zimprich
- J1: value I2C_1 -> I2C0_1; footprint Connector_PinHeader_2.54mm:PinHeader_1x04_P2.54mm_Vertical -> Connector_JST:JST_XH_B4B-XH-A_1x04_P2.50mm_Vertical
- J2: value I2C_2 -> I2C0_2; footprint Connector_PinHeader_2.54mm:PinHeader_1x04_P2.54mm_Vertical -> Connector_JST:JST_XH_B4B-XH-A_1x04_P2.50mm_Vertical
- J25: value TX0/RX0 -> Ser0
- J26: value TX1/RX1 -> Ser1
- J27: value TX2/RX2 -> Ser2
- J28: value GPS_TX/GPS_RX -> Ser3
- J3: value I2C_3 -> I2C1_1; footprint Connector_PinHeader_2.54mm:PinHeader_1x04_P2.54mm_Vertical -> Connector_JST:JST_XH_B4B-XH-A_1x04_P2.50mm_Vertical
- J6, J7, J8, J9: footprint Connector_PinHeader_2.54mm:PinHeader_1x03_P2.54mm_Vertical -> Connector_JST:JST_XH_B3B-XH-A_1x03_P2.50mm_Vertical
- XA1: symbol arduino:Arduino_Due_Shield -> Ardumower-rescue:Arduino_Due_Shield-arduino
Connections:
- net labels added: RX3, TX3, freePinD42, freePinD43, pinMotorMow1Sense, pinMotorMow2Sense
- net labels removed: GPS_RX, GPS_TX, pinLawnBackRecv, pinLawnBackSend, pinMotorLeftSense2, pinMotorMowSense, pinPerimeterCenter
- wire segments 87 -> 75
- no-connect marks 4 -> 2
Other:
- moved on the sheet: J20, J25, J28, J7, R14, R17, R18

Commit message: half job
Parts:
- removed J27: Ser2, Connector_PinHeader_2.54mm:PinHeader_1x05_P2.54mm_Vertical, symbol Connector:Screw_Terminal_01x05
- removed J8: Tilt, Connector_JST:JST_XH_B3B-XH-A_1x03_P2.50mm_Vertical, symbol Connector:Screw_Terminal_01x03
- removed R1, R2, R5: 1KO, Resistor_THT:R_Axial_DIN0207_L6.3mm_D2.5mm_P2.54mm_Vertical, symbol Device:R
- removed R12, R6, R7: 2KO, Resistor_THT:R_Axial_DIN0207_L6.3mm_D2.5mm_P2.54mm_Vertical, symbol Device:R
- added J11: Sonar_C, Connector_JST:JST_XH_B4B-XH-A_1x04_P2.50mm_Vertical, symbol Connector:Screw_Terminal_01x04
- added J8: Tilt, Connector_JST:JST_XH_B2B-XH-A_1x02_P2.50mm_Vertical, symbol Connector:Screw_Terminal_01x02
- J12, J13: footprint Connector_PinHeader_2.54mm:PinHeader_1x03_P2.54mm_Vertical -> Connector_JST:JST_XH_B3B-XH-A_1x03_P2.50mm_Vertical
- J14, J16: footprint Connector_PinHeader_2.54mm:PinHeader_1x04_P2.54mm_Vertical -> Connector_JST:JST_XH_B4B-XH-A_1x04_P2.50mm_Vertical
- J15: value Sonar_C -> Ser2 ESP32; footprint Connector_PinHeader_2.54mm:PinHeader_1x04_P2.54mm_Vertical -> Connector_JST:JST_XH_B4B-XH-A_1x04_P2.50mm_Vertical
- J20: footprint Zimprich:Pin_Header_KK110_1x02_3D -> Connector_JST:JST_XH_B2B-XH-A_1x02_P2.50mm_Vertical
- J25, J26, J28: footprint Connector_PinHeader_2.54mm:PinHeader_1x05_P2.54mm_Vertical -> Connector_JST:JST_XH_B5B-XH-A_1x05_P2.50mm_Vertical
Connections:
- net +3V3: now also J14.1 (Pin_1), J16.1 (Pin_1), J11.1 (Pin_1); no longer J25.1 (Pin_1)
- net +5V: no longer J14.1 (Pin_1), J15.1 (Pin_1), J16.1 (Pin_1), J25.5 (Pin_5)
- net +9V: now also J15.4 (Pin_4)
- net GND: now also J15.1 (Pin_1), J11.2 (Pin_2), J8.1 (Pin_1); no longer J15.2 (Pin_2), J25.2 (Pin_2)
- net RX0: no longer J25.3 (Pin_3)
- net RX2: now also J15.2 (Pin_2)
- net TX0: no longer J25.4 (Pin_4)
- net TX2: now also J15.3 (Pin_3)
- net pinSonarCenterEcho: now also J11.3 (Pin_3)
- net pinSonarCenterTrigger: now also J11.4 (Pin_4); no longer J15.4 (Pin_4)
- net pinSonarLeftEcho: now also J16.3 (Pin_3)
- net pinSonarRightEcho: now also J14.3 (Pin_3)
- net pinTilt: now also J8.2 (Pin_2)
Other:
- moved on the sheet: J1, J16, J17, J18, J19, J2, J22, J23, J3, J4, J9, R13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
